File: hardware/pcb/i2c.kicad_sch (KiCad schematic)
At the start: 17 parts, among them U10 AS7341-DLGM, U11 TMP117AIDRVR, U12 MLX90632SLD-DCB-000-RE, U13 BME280, U14 LSM6DSV80XTR, U9 PCA9306DCUR

Commit message: Use official CAD and shrink the hw_v1 board to 37x30 mm.
Replace the hand-drawn AFE4900, AD5940, ADS1292R, AS7341, MLX90632,
TMP117, LSM6DSV80X, and MCP73831 symbols and footprints with the
SnapMagic and Ultra Librarian libraries. ADS1292R is now the QFN-32
ADS1292RIRSMT, and MLX90632SLD-DCB-100-SP moves SDA/SCL onto the
existing 1.8 V bus. Pin headers and mounting holes are flat solder
pads. The unrouted 4-layer placement keeps the antenna on the left
edge and the skin sensors together on the bottom.

Co-authored-by: Riyu-D1 <Riyu-D1@users.noreply.github.com>
Parts:
- removed U10: AS7341-DLGM, Package_LGA:AMS_OLGA-8_2x3.1mm_P0.8mm, symbol vitalq:AS7341DLG
- removed U12: MLX90632SLD-DCB-000-RE, vitalq:MLX90632, symbol vitalq:MLX90632
- removed U14: LSM6DSV80XTR, vitalq:LSM6DSV80X, symbol vitalq:LSM6DSV80X
- added U10: AS7341-DLGM, snap:AS7341DLGT, symbol vitalq:AS7341-DLGM
- added U12: MLX90632SLD-DCB-100-SP, snap:MLX90632SLDDCB100SP, symbol vitalq:MLX90632SLD-DCB-100-SP
- added U14: LSM6DSV80XTR, snap:QFN_LSM6DSV80XTR_STM, symbol vitalq:LSM6DSV80XTR
- U11: footprint Package_SON:WSON-6-1EP_2x2mm_P0.65mm_EP1x1.6mm -> snap:SON65P200X200X80-7N
Connections:
- net +1V8: now also U10.1 (VDD)
- net +3V3: now also U11.5 (V+), U12.2 (VDD), U14.12, U14.5, U14.8; no longer U11.4 (V+)
- net GND: now also U11.4 (ADD0), U10.3 (GND), U10.5 (PGND), U12.3 (GND), U12.5 (ADDR), U12.6 (EP), U14.1, U14.2, U14.3, U14.6, U14.7; no longer U11.3 (ADD0)
- net I2C_SCL: now also U14.13
- net I2C_SCL_1V8: now also U10.2 (SCL), U12.4 (SCL)
- net I2C_SDA: now also U14.14
- net I2C_SDA_1V8: now also U10.8 (SDA), U12.1 (SDA)
- net LSM6_INT1: now also U14.4
- net TMP117_ALERT: now also U11.3 (ALERT); no longer U11.5 (ALERT)
Other:
- note added: "MLX90632SLD-DCB-100-SP is the 1.8 V I2C option. VDD is still 3.3 V. ADDR = GND is 0x3A."
- note removed: "MLX90632 0x3A, ADDR = GND"

Commit message: Add the chest-board sensors and replace the 3.3 V LDO with a TPS63802.
The unrouted 40 x 34 mm board keeps every previous part except the off-board PPG pads, which the SFH 7072 replaces. Respiration, a second ECG lead, electrode protection, EDA, fuel gauge, flash, and the I/O expander are in the schematic.

Co-authored-by: Riyu-D1 <Riyu-D1@users.noreply.github.com>
Parts:
- added C61: 100n, Capacitor_SMD:C_0402_1005Metric, symbol vitalq:C
- added D10: NF2W757G-F1, vitalq:NF2W757G, symbol vitalq:LED_AK
- added D11: SFH4053, LED_SMD:LED_0402_1005Metric, symbol vitalq:LED_AK
- added Q1: CSD13380F3, Package_DFN_QFN:Texas_PicoStar_DFN-3_0.69x0.60mm, symbol vitalq:CSD13380F3
- added R47: 100, Resistor_SMD:R_0402_1005Metric, symbol vitalq:R
- added R48: 100k, Resistor_SMD:R_0402_1005Metric, symbol vitalq:R
- added U20: TMP117AIDRVR, snap:SON65P200X200X80-7N, symbol vitalq:TMP117AIDRVR
Connections:
- net +3V3: now also C61.1, D10.1 (A), R47.1, U20.4 (ADD0), U20.5 (V+)
- net GND: now also C61.2, Q1.2 (S), R48.2, U20.2 (GND_1), U20.7 (GND_2)
- net I2C_SCL: now also U20.1 (SCL)
- net I2C_SDA: now also U20.6 (SDA)
- net LDR: now reaches U10.4 (LDR)
- net LDR: now also D10.2 (K)
- new net IR_AN: D11.1 (A), R47.2
- new net IR_GATE: Q1.1 (G), R48.1
- new net IR_K: D11.2 (K), Q1.3 (D)
Other:
- note added: "AS7341 0x39 at 1.8 V. D10 anode is +3V3, never VBAT. LDR abs max is 3.6 V."
- note added: "TMP117 U11 0x48, ADD0 = GND"
- note added: "U20 is the second TMP117, ADD0 = +3V3, address 0x49."
- note removed: "AS7341 address 0x39. VDD 1.8 V. LDR and LED pins open."
- note removed: "TMP117 0x48, ADD0 = GND"

Commit message: Fix the CP2102N sense pin and add electrode creepage slots.
The USB sense pin was tied to 5 V. It now uses the datasheet divider, with the reset pull-up and the missing 100 nF bypasses. The TMP117 alert has its pull-up. Three slots raise creepage between the pulse resistors to 4.0 mm on a 1.6 mm board. Nothing was removed.

Co-authored-by: Riyu-D1 <Riyu-D1@users.noreply.github.com>
Parts:
- added R65: 10k, Resistor_SMD:R_0402_1005Metric, symbol vitalq:R
Connections:
- net +3V3: now also R65.1
- net TMP117_ALERT: now also R65.2
Other:
- note added: "TMP117 U11 0x48, ADD0 = GND. R65 pulls ALERT up."
- note removed: "TMP117 U11 0x48, ADD0 = GND"
