File: hardware/pcb/i2c.kicad_sch (KiCad schematic)
At the start: 26 parts, among them Q1 CSD13380F3T, U10 AS7341-DLGM, U11 TMP117AIDRVR, U12 MLX90632SLD-DCB-100-SP, U13 BME280, U14 LSM6DSV80XTR, U20 TMP117AIDRVR, U9 PCA9306DCUR

Commit message: Improve hw_v2 PCB: HV tail chains, decoupling re-park, power islands, U22 escape
Schematic fixes:
- Fix SWEAT_RE silently shorted to GND (D27 pin-endpoint collision)
- Fix L2/TX_5V boost miswire (VBAT_SYS->TX_SW, rail was dead)
- Add J11/J13 HV-boundary chains: R118-R122 2512 cut-points + D26-D30 DNP TPD clamps
- Correct J12 to FH12-14S-0.5SH land; R114 LED_AN fed from TX_5V
- Move U24 VBACKUP to dedicated RTC_VBK net; ADS1292 CLK grounded
- Add CS pull-ups (R115-R117), TP28, C84 (U4 +3V3 input decoupling)
- New hw_v2 parts: U22 MAX86178, U23 SHT45, U24 RTC (DNP), U25 IM69D130 (DNP),
  D12 SFH4735 NIR + Q4 gate, J9-J13 tails

Layout:
- Grow board 32->40 mm east; five 2512 HV parts could not fit at 32 mm
- Re-park ~30 decoupling passives adjacent to their ICs
- Replace phantom moat wall slots with a real >=1.0 mm channel
- Own-layer pour keepouts under HV pads; wider stitch-via HV margin
- U22 WLP: drop 28 NC lands (rows B-E) to open B.Cu escape for F-row
- Retarget dead power islands (TX_5V over its 9 loads, +1V8 under LDO, +3V3 at U7)

BOM/CPL: footprint-aware 0R mapping (0402->C17168, 2512->C2908946),
DNP parts excluded, J11/J13 pads DNP'd, U1 MPN corrected.

Gates: placement zero (291 parts), ERC 0, DRC non-unrouted 0
(9 inherent Q1/Q2/Q4 intra-package clearances waived-by-name).
Board remains unrouted by design - research prototype, not fab-ready.

Generated with [Devin](https://devin.ai)

Co-Authored-By: Devin <158243242+devin-ai-integration[bot]@users.noreply.github.com>
Parts:
- added C76, C77: 100n, Capacitor_SMD:C_0402_1005Metric, symbol vitalq:C
- added D12: SFH 4735 730nm, LED_SMD:LED_0402_1005Metric, symbol vitalq:LED_AK
- added Q4: CSD13380F3T, Package_DFN_QFN:Texas_PicoStar_DFN-3_0.69x0.60mm, symbol vitalq:CSD13380F3
- added R109: 100, Resistor_SMD:R_0402_1005Metric, symbol vitalq:R
- added R110: 100k, Resistor_SMD:R_0402_1005Metric, symbol vitalq:R
- added R112, R115: 10k, Resistor_SMD:R_0402_1005Metric, symbol vitalq:R
- added U23: SHT45-AD1B, vitalq:SHT45_DFN4, symbol vitalq:SHT45-AD1B
- added U24: RV-3028-C7, vitalq:RV3028C7, symbol vitalq:RV-3028-C7
Connections:
- net +3V3: now also C76.1, C77.1, R109.1, R112.1, U23.3 (VDD), U24.7 (VDD)
- net GND: now also C76.2, C77.2, Q4.2 (S), R110.2, R115.2, U23.4 (VSS), U24.5 (VSS), U24.8 (EVI)
- net I2C_SCL: now also U23.2 (SCL), U24.3 (SCL)
- net I2C_SDA: now also U23.1 (SDA), U24.4 (SDA)
- new net NIR730_GATE: Q4.1 (G), R110.1
- new net NIR_AN: D12.1 (A), R109.2
- new net NIR_K: D12.2 (K), Q4.3 (D)
- new net RTC_INT: R112.2, U24.2 (INT)
- new net RTC_VBK: R115.1, U24.6 (VBACKUP)
- no-connect marks 4 -> 5
Other:
- note added: "D12 is the 730 nm LED; Q4 gate is AD5940 GPIO2 (E1). Pairs with the AS7341 NIR channel."
- note added: "U23 SHT45-AD1B, 0x44, skin side."
- note added: "U24 RV-3028-C7, DNP, 0x52. VBACKUP to VSS via R115 10k; CLKOUT open."
