File: hardware/pcb/i2c.kicad_sch (KiCad schematic)
At the start: 36 parts, among them Q1 CSD13380F3T, Q4 CSD13380F3T, U10 AS7341-DLGM, U11 TMP117AIDRVR, U12 MLX90632SLD-DCB-100-SP, U13 BME280, U14 LSM6DSV80XTR, U20 TMP117AIDRVR, U23 SHT45-AD1B, U24 RV-3028-C7, U9 PCA9306DCUR

Commit message: Fit tier-1 DNP parts: U24 RTC, U25 mic, D26-D30 tail clamps
- U24 RV-3028-C7 + C77/R112/R115 support passives now fitted
- U25 IM69D130 PDM mic + C78 decoupling now fitted
- D26-D30 TPD1E10B06 tail ESD clamps now fitted
- remaining DNP are intentional options only: R61 cell-NTC,
  R104/R105 CP2102 USB strap, R107/R108 SPARE divider, J12, J13

check.sh PASS: ERC 0; gates 0; DRC = 499 unrouted items only.

Generated with [Devin](https://devin.ai)

Co-Authored-By: Devin <158243242+devin-ai-integration[bot]@users.noreply.github.com>
Parts:
- C77, R112, R115, U24: now fitted
Other:
- note added: "U24 RV-3028-C7, 0x52. VBACKUP to VSS via R115 10k; CLKOUT open."
- note removed: "U24 RV-3028-C7, DNP, 0x52. VBACKUP to VSS via R115 10k; CLKOUT open."
