File: hardware/pcb/usb.kicad_sch (KiCad schematic)
At the start: 8 parts, among them U5 CP2102N-A02-GQFN28R

Commit message: Fix the review's datasheet errors without changing respiration or the GDTs.
Replace the MCP73831 with a BQ25170 so a flat cell still charges from USB, add the missing series protection and ESP32/CP2102 passives, and withdraw the claim that respiration still works with 51 kΩ in the loop.

Co-authored-by: Riyu-D1 <Riyu-D1@users.noreply.github.com>
Parts:
- added Q3: BC847BS,115, Package_TO_SOT_SMD:SOT-363_SC-70-6, symbol vitalq:BC847BS_DUAL
- added R70, R71: 10k, Resistor_SMD:R_0402_1005Metric, symbol vitalq:R
- added R72, R73: 1k, Resistor_SMD:R_0402_1005Metric, symbol vitalq:R
Connections:
- net ESP_RX: now also R73.2; no longer U5.26 (TXD)
- net ESP_TX: now also R72.1; no longer U5.25 (RXD)
- net CP_RTS: now reaches U5.24 (~{RTS})
- net CP_RTS: now also Q3.1 (E1), R71.1
- net CP_DTR: now reaches U5.28 (~{DTR})
- net CP_DTR: now also Q3.4 (E2), R70.1
- new net CP_RX: R72.2, U5.25 (RXD)
- new net CP_TX: R73.1, U5.26 (TXD)
- new net ESP_EN: Q3.6 (C1)
- new net ESP_IO0: Q3.3 (C2)
- new net Q3_B1: Q3.2 (B1), R70.2
- new net Q3_B2: Q3.5 (B2), R71.2
- no-connect marks 14 -> 12
Other:
- note added: "Q3 is the DevKitC auto-program pair: DTR/RTS to EN and GPIO0. R70 and R71 are the 10k bases."
- note added: "R72 and R73 are 1k in series with TX and RX so an unpowered side is not back-driven."

Commit message: Prepare hw_v1 for prefab review without claiming the route is finished.
Add the gauge TDFN, USB ESD, sense links, test access, and JLC BOM fields, and keep the partial Freerouting result with the remaining open nets listed.

Co-authored-by: Riyu-D1 <Riyu-D1@users.noreply.github.com>
Parts:
- C10: footprint Capacitor_SMD:C_0402_1005Metric -> Capacitor_SMD:C_0603_1608Metric
Changed lines of the file:
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@@
 		(instances
 			(project "vitalq_hw_v1"
-				(path "/a3eebb51-17e8-4aa6-8fe3-3d57dec01ed3/e6e91e9e-59d1-4f2e-9de6-0b31256d1bd9"
+				(path "/c5177a17-7f1f-4b29-a2a6-55306503fc64/ee2bc8d8-e754-4dce-ac55-2b68f03a01f9"
 					(reference "U5")
 					(unit 1)
@@
 		(on_board no)
 		(dnp no)
-		(property "Reference" "#PWR040"
+		(property "Reference" "#PWR039"
 			(at 179.07 84.56 0)
 			(effects (font (size 1.27 1.27)) (hide yes))
@@
 		(instances
 			(project "vitalq_hw_v1"
-				(path "/a3eebb51-17e8-4aa6-8fe3-3d57dec01ed3/e6e91e9e-59d1-4f2e-9de6-0b31256d1bd9"
-					(reference "#PWR040")
+				(path "/c5177a17-7f1f-4b29-a2a6-55306503fc64/ee2bc8d8-e754-4dce-ac55-2b68f03a01f9"
+					(reference "#PWR039")
 					(unit 1)
 				)
@@
 		(on_board no)
 		(dnp no)
-		(property "Reference" "#PWR041"
+		(property "Reference" "#PWR040"
 			(at 199.39 167.11 0)
 			(effects (font (size 1.27 1.27)) (hide yes))
@@
 		(instances
 			(project "vitalq_hw_v1"
-				(path "/a3eebb51-17e8-4aa6-8fe3-3d57dec01ed3/e6e91e9e-59d1-4f2e-9de6-0b31256d1bd9"
-					(reference "#PWR041")
+				(path "/c5177a17-7f1f-4b29-a2a6-55306503fc64/ee2bc8d8-e754-4dce-ac55-2b68f03a01f9"
+					(reference "#PWR040")
 					(unit 1)
 				)
@@
 		(instances
 			(project "vitalq_hw_v1"
-				(path "/a3eebb51-17e8-4aa6-8fe3-3d57dec01ed3/e6e91e9e-59d1-4f2e-9de6-0b31256d1bd9"
+				(path "/c5177a17-7f1f-4b29-a2a6-55306503fc64/ee2bc8d8-e754-4dce-ac55-2b68f03a01f9"
 					(reference "C9")
 					(unit 1)
@@
 		(on_board no)
 		(dnp no)
-		(property "Reference" "#PWR042"
+		(property "Reference" "#PWR041"
 			(at 54.61 75.67 0)
 			(effects (font (size 1.27 1.27)) (hide yes))
@@
 		(instances
 			(project "vitalq_hw_v1"
-				(path "/a3eebb51-17e8-4aa6-8fe3-3d57dec01ed3/e6e91e9e-59d1-4f2e-9de6-0b31256d1bd9"
-					(reference "#PWR042")
+				(path "/c5177a17-7f1f-4b29-a2a6-55306503fc64/ee2bc8d8-e754-4dce-ac55-2b68f03a01f9"
+					(reference "#PWR041")
 					(unit 1)
 				)
@@
 		(instances
 			(project "vitalq_hw_v1"
-				(path "/a3eebb51-17e8-4aa6-8fe3-3d57dec01ed3/e6e91e9e-59d1-4f2e-9de6-0b31256d1bd9"
+				(path "/c5177a17-7f1f-4b29-a2a6-55306503fc64/ee2bc8d8-e754-4dce-ac55-2b68f03a01f9"
 					(reference "C62")
 					(unit 1)
@@
 		(on_board no)
 		(dnp no)
-		(property "Reference" "#PWR043"
+		(property "Reference" "#PWR042"
 			(at 77.47 106.15 0)
 			(effects (font (size 1.27 1.27)) (hide yes))
@@
 		(instances
 			(project "vitalq_hw_v1"
-				(path "/a3eebb51-17e8-4aa6-8fe3-3d57dec01ed3/e6e91e9e-59d1-4f2e-9de6-0b31256d1bd9"
-					(reference "#PWR043")
+				(path "/c5177a17-7f1f-4b29-a2a6-55306503fc64/ee2bc8d8-e754-4dce-ac55-2b68f03a01f9"
+					(reference "#PWR042")
 					(unit 1)
 				)
@@
 			(effects (font (size 1.27 1.27)))
 		)
-		(property "Footprint" "Capacitor_SMD:C_0402_1005Metric"
+		(property "Footprint" "Capacitor_SMD:C_0603_1608Metric"
 			(at 100.33 69.85 0)
 			(effects (font (size 1.27 1.27)) (hide yes))
@@
 		(instances
 			(project "vitalq_hw_v1"
-				(path "/a3eebb51-17e8-4aa6-8fe3-3d57dec01ed3/e6e91e9e-59d1-4f2e-9de6-0b31256d1bd9"
+				(path "/c5177a17-7f1f-4b29-a2a6-55306503fc64/ee2bc8d8-e754-4dce-ac55-2b68f03a01f9"
 					(reference "C10")
 					(unit 1)
@@
 		(on_board no)
 		(dnp no)
-		(property "Reference" "#PWR044"
+		(property "Reference" "#PWR043"
 			(at 100.33 60.43 0)
 			(effects (font (size 1.27 1.27)) (hide yes))
@@
 		(instances
 			(project "vitalq_hw_v1"
-				(path "/a3eebb51-17e8-4aa6-8fe3-3d57dec01ed3/e6e91e9e-59d1-4f2e-9de6-0b31256d1bd9"
-					(reference "#PWR044")
+				(path "/c5177a17-7f1f-4b29-a2a6-55306503fc64/ee2bc8d8-e754-4dce-ac55-2b68f03a01f9"
+					(reference "#PWR043")
 					(unit 1)
 				)
@@
 		(on_board no)
 		(dnp no)
-		(property "Reference" "#PWR045"
+		(property "Reference" "#PWR044"
 			(at 100.33 75.67 0)
 			(effects (font (size 1.27 1.27)) (hide yes))
@@
 		(instances
 			(project "vitalq_hw_v1"
-				(path "/a3eebb51-17e8-4aa6-8fe3-3d57dec01ed3/e6e91e9e-59d1-4f2e-9de6-0b31256d1bd9"
-					(reference "#PWR045")
+				(path "/c5177a17-7f1f-4b29-a2a6-55306503fc64/ee2bc8d8-e754-4dce-ac55-2b68f03a01f9"
+					(reference "#PWR044")
 					(unit 1)
 				)
@@
 		(instances
 			(project "vitalq_hw_v1"
-				(path "/a3eebb51-17e8-4aa6-8fe3-3d57dec01ed3/e6e91e9e-59d1-4f2e-9de6-0b31256d1bd9"
+				(path "/c5177a17-7f1f-4b29-a2a6-55306503fc64/ee2bc8d8-e754-4dce-ac55-2b68f03a01f9"
 					(reference "C63")
 					(unit 1)
@@
 		(on_board no)
 		(dnp no)
-		(property "Reference" "#PWR046"
+		(property "Reference" "#PWR045"
 			(at 121.92 60.43 0)
 			(effects (font (size 1.27 1.27)) (hide yes))
@@
 		(instances
 			(project "vitalq_hw_v1"
-				(path "/a3eebb51-17e8-4aa6-8fe3-3d57dec01ed3/e6e91e9e-59d1-4f2e-9de6-0b31256d1bd9"
-					(reference "#PWR046")
+				(path "/c5177a17-7f1f-4b29-a2a6-55306503fc64/ee2bc8d8-e754-4dce-ac55-2b68f03a01f9"
+					(reference "#PWR045")
 					(unit 1)
 				)
@@
 		(on_board no)
 		(dnp no)
-		(property "Reference" "#PWR047"
+		(property "Reference" "#PWR046"
 			(at 121.92 75.67 0)
 			(effects (font (size 1.27 1.27)) (hide yes))
@@
 		(instances
 			(project "vitalq_hw_v1"
-				(path "/a3eebb51-17e8-4aa6-8fe3-3d57dec01ed3/e6e91e9e-59d1-4f2e-9de6-0b31256d1bd9"
-					(reference "#PWR047")
+				(path "/c5177a17-7f1f-4b29-a2a6-55306503fc64/ee2bc8d8-e754-4dce-ac55-2b68f03a01f9"
+					(reference "#PWR046")
 					(unit 1)
 				)
@@
 		(instances
 			(project "vitalq_hw_v1"
-				(path "/a3eebb51-17e8-4aa6-8fe3-3d57dec01ed3/e6e91e9e-59d1-4f2e-9de6-0b31256d1bd9"
+				(path "/c5177a17-7f1f-4b29-a2a6-55306503fc64/ee2bc8d8-e754-4dce-ac55-2b68f03a01f9"
 					(reference "R62")
 					(unit 1)
@@
 		(instances
 			(project "vitalq_hw_v1"
-				(path "/a3eebb51-17e8-4aa6-8fe3-3d57dec01ed3/e6e91e9e-59d1-4f2e-9de6-0b31256d1bd9"
+				(path "/c5177a17-7f1f-4b29-a2a6-55306503fc64/ee2bc8d8-e754-4dce-ac55-2b68f03a01f9"
 					(reference "R63")
 					(unit 1)
@@
 		(on_board no)
 		(dnp no)
-		(property "Reference" "#PWR048"
+		(property "Reference" "#PWR047"
 			(at 54.61 135.36 0)
 			(effects (font (size 1.27 1.27)) (hide yes))
@@
 		(instances
 			(project "vitalq_hw_v1"
-				(path "/a3eebb51-17e8-4aa6-8fe3-3d57dec01ed3/e6e91e9e-59d1-4f2e-9de6-0b31256d1bd9"
-					(reference "#PWR048")
+				(path "/c5177a17-7f1f-4b29-a2a6-55306503fc64/ee2bc8d8-e754-4dce-ac55-2b68f03a01f9"
+					(reference "#PWR047")
 					(unit 1)
 				)
@@
 		(instances
 			(project "vitalq_hw_v1"
-				(path "/a3eebb51-17e8-4aa6-8fe3-3d57dec01ed3/e6e91e9e-59d1-4f2e-9de6-0b31256d1bd9"
+				(path "/c5177a17-7f1f-4b29-a2a6-55306503fc64/ee2bc8d8-e754-4dce-ac55-2b68f03a01f9"
 					(reference "R64")
 					(unit 1)
@@
 		(on_board no)
 		(dnp no)
-		(property "Reference" "#PWR049"
+		(property "Reference" "#PWR048"
 			(at 90.17 150.6 0)
 			(effects (font (size 1.27 1.27)) (hide yes))
@@
 		(instances
 			(project "vitalq_hw_v1"
-				(path "/a3eebb51-17e8-4aa6-8fe3-3d57dec01ed3/e6e91e9e-59d1-4f2e-9de6-0b31256d1bd9"
-					(reference "#PWR049")
+				(path "/c5177a17-7f1f-4b29-a2a6-55306503fc64/ee2bc8d8-e754-4dce-ac55-2b68f03a01f9"
+					(reference "#PWR048")
 					(unit 1)
 				)
@@
 		(instances
 			(project "vitalq_hw_v1"
-				(path "/a3eebb51-17e8-4aa6-8fe3-3d57dec01ed3/e6e91e9e-59d1-4f2e-9de6-0b31256d1bd9"
+				(path "/c5177a17-7f1f-4b29-a2a6-55306503fc64/ee2bc8d8-e754-4dce-ac55-2b68f03a01f9"
 					(reference "R72")
 					(unit 1)
@@
 		(instances
 			(project "vitalq_hw_v1"
-				(path "/a3eebb51-17e8-4aa6-8fe3-3d57dec01ed3/e6e91e9e-59d1-4f2e-9de6-0b31256d1bd9"
+				(path "/c5177a17-7f1f-4b29-a2a6-55306503fc64/ee2bc8d8-e754-4dce-ac55-2b68f03a01f9"
 					(reference "R73")
 					(unit 1)
@@
 		(instances
 			(project "vitalq_hw_v1"
-				(path "/a3eebb51-17e8-4aa6-8fe3-3d57dec01ed3/e6e91e9e-59d1-4f2e-9de6-0b31256d1bd9"
+				(path "/c5177a17-7f1f-4b29-a2a6-55306503fc64/ee2bc8d8-e754-4dce-ac55-2b68f03a01f9"
 					(reference "Q3")
 					(unit 1)
@@
 		(instances
 			(project "vitalq_hw_v1"
-				(path "/a3eebb51-17e8-4aa6-8fe3-3d57dec01ed3/e6e91e9e-59d1-4f2e-9de6-0b31256d1bd9"
+				(path "/c5177a17-7f1f-4b29-a2a6-55306503fc64/ee2bc8d8-e754-4dce-ac55-2b68f03a01f9"
 					(reference "R70")
 					(unit 1)
@@
 		(instances
 			(project "vitalq_hw_v1"
-				(path "/a3eebb51-17e8-4aa6-8fe3-3d57dec01ed3/e6e91e9e-59d1-4f2e-9de6-0b31256d1bd9"
+				(path "/c5177a17-7f1f-4b29-a2a6-55306503fc64/ee2bc8d8-e754-4dce-ac55-2b68f03a01f9"
 					(reference "R71")
 					(unit 1)
@@
 		(on_board no)
 		(dnp no)
-		(property "Reference" "#FLG050"
+		(property "Reference" "#FLG049"
 			(at 142.24 60.43 0)
 			(effects (font (size 1.27 1.27)) (hide yes))
@@
 		(instances
 			(project "vitalq_hw_v1"
-				(path "/a3eebb51-17e8-4aa6-8fe3-3d57dec01ed3/e6e91e9e-59d1-4f2e-9de6-0b31256d1bd9"
-					(reference "#FLG050")
-					(unit 1)
-				)
+				(path "/c5177a17-7f1f-4b29-a2a6-55306503fc64/ee2bc8d8-e754-4dce-ac55-2b68f03a01f9"
+					(reference "#FLG049")
+					(unit 1)
+				)
