File: hardware/pcb/usb.kicad_sch (KiCad schematic)
At the start: 13 parts, among them Q3 BC847BS,115, U5 CP2102N-A02-GQFN28R

Commit message: Improve hw_v2 PCB: HV tail chains, decoupling re-park, power islands, U22 escape
Schematic fixes:
- Fix SWEAT_RE silently shorted to GND (D27 pin-endpoint collision)
- Fix L2/TX_5V boost miswire (VBAT_SYS->TX_SW, rail was dead)
- Add J11/J13 HV-boundary chains: R118-R122 2512 cut-points + D26-D30 DNP TPD clamps
- Correct J12 to FH12-14S-0.5SH land; R114 LED_AN fed from TX_5V
- Move U24 VBACKUP to dedicated RTC_VBK net; ADS1292 CLK grounded
- Add CS pull-ups (R115-R117), TP28, C84 (U4 +3V3 input decoupling)
- New hw_v2 parts: U22 MAX86178, U23 SHT45, U24 RTC (DNP), U25 IM69D130 (DNP),
  D12 SFH4735 NIR + Q4 gate, J9-J13 tails

Layout:
- Grow board 32->40 mm east; five 2512 HV parts could not fit at 32 mm
- Re-park ~30 decoupling passives adjacent to their ICs
- Replace phantom moat wall slots with a real >=1.0 mm channel
- Own-layer pour keepouts under HV pads; wider stitch-via HV margin
- U22 WLP: drop 28 NC lands (rows B-E) to open B.Cu escape for F-row
- Retarget dead power islands (TX_5V over its 9 loads, +1V8 under LDO, +3V3 at U7)

BOM/CPL: footprint-aware 0R mapping (0402->C17168, 2512->C2908946),
DNP parts excluded, J11/J13 pads DNP'd, U1 MPN corrected.

Gates: placement zero (291 parts), ERC 0, DRC non-unrouted 0
(9 inherent Q1/Q2/Q4 intra-package clearances waived-by-name).
Board remains unrouted by design - research prototype, not fab-ready.

Generated with [Devin](https://devin.ai)

Co-Authored-By: Devin <158243242+devin-ai-integration[bot]@users.noreply.github.com>
Parts:
- added R102, R103, R104, R105: 0, Resistor_SMD:R_0402_1005Metric, symbol vitalq:R
Connections:
- net USB_DM: now also R103.1, R105.1; no longer U5.5 (D-)
- net USB_DP: now also R102.1, R104.1; no longer U5.4 (D+)
- new net USB_DM_CP: R105.2, U5.5 (D-)
- new net USB_DM_S3: R103.2
- new net USB_DP_CP: R104.2, U5.4 (D+)
- new net USB_DP_S3: R102.2
Other:
- note added: "Alternate strap (DNP): move 0R to R104/R105 for the CP2102 bridge."
- note added: "Fitted: J1 -> S3 IO20/IO19 (native USB, on-chip JTAG+console)."
- note added: "U5/U21/Q3 are unchanged. CP2102 keeps UART0 on ESP_TX/ESP_RX."
- note added: "USB D+/D- strap links"
