File: hardware/pcb/vitalq_hw_v1.kicad_sch (KiCad schematic)
At the start: 29 parts, among them J1 USB-C, J2 LiPo pads, Q2 CSD13380F3T, U17 MAX17048G+T10, U2 BQ25170DSGR, U3 TPS63802DLAR, U4 TPS7A2018PDBVR

Commit message: Improve hw_v2 PCB: HV tail chains, decoupling re-park, power islands, U22 escape
Schematic fixes:
- Fix SWEAT_RE silently shorted to GND (D27 pin-endpoint collision)
- Fix L2/TX_5V boost miswire (VBAT_SYS->TX_SW, rail was dead)
- Add J11/J13 HV-boundary chains: R118-R122 2512 cut-points + D26-D30 DNP TPD clamps
- Correct J12 to FH12-14S-0.5SH land; R114 LED_AN fed from TX_5V
- Move U24 VBACKUP to dedicated RTC_VBK net; ADS1292 CLK grounded
- Add CS pull-ups (R115-R117), TP28, C84 (U4 +3V3 input decoupling)
- New hw_v2 parts: U22 MAX86178, U23 SHT45, U24 RTC (DNP), U25 IM69D130 (DNP),
  D12 SFH4735 NIR + Q4 gate, J9-J13 tails

Layout:
- Grow board 32->40 mm east; five 2512 HV parts could not fit at 32 mm
- Re-park ~30 decoupling passives adjacent to their ICs
- Replace phantom moat wall slots with a real >=1.0 mm channel
- Own-layer pour keepouts under HV pads; wider stitch-via HV margin
- U22 WLP: drop 28 NC lands (rows B-E) to open B.Cu escape for F-row
- Retarget dead power islands (TX_5V over its 9 loads, +1V8 under LDO, +3V3 at U7)

BOM/CPL: footprint-aware 0R mapping (0402->C17168, 2512->C2908946),
DNP parts excluded, J11/J13 pads DNP'd, U1 MPN corrected.

Gates: placement zero (291 parts), ERC 0, DRC non-unrouted 0
(9 inherent Q1/Q2/Q4 intra-package clearances waived-by-name).
Board remains unrouted by design - research prototype, not fab-ready.

Generated with [Devin](https://devin.ai)

Co-Authored-By: Devin <158243242+devin-ai-integration[bot]@users.noreply.github.com>
Parts:
- added C84: 1u, Capacitor_SMD:C_0402_1005Metric, symbol vitalq:C
Connections:
- net +3V3: now also C84.1
- net GND: now also J1.SH (SHIELD), C84.2; no longer J1.S1 (SHIELD)
Other:
- added sheet MAX86178 and tails (max86178.kicad_sch)
