File: hardware/pcb/vitalq_hw_v1.kicad_sch (KiCad schematic)
At the start: 30 parts, among them J1 USB-C, J2 LiPo pads, Q2 CSD13380F3T, U17 MAX17048G+T10, U2 BQ25170DSGR, U3 TPS63802DLAR, U4 TPS7A2018PDBVR

Commit message: Add C85 47uF VBAT bulk cap at battery input
Stress-test finding: VBAT bulk was ~10-15 uF total (C2 4.7u + C58 100n).
WiFi TX bursts (~300-500 mA) + LED pulses could sag a small LiPo.

- C85 CL10A476MQ8NRNC (0603, 47 uF 6.3V X5R, LCSC C19702) on VBAT
- Placed bottom side at (2.3, 22.5), ~11 mm from J2 battery pads

parts 291 -> 292. Gates: clashes 0 / edge 0 / pth 0 / pad-miss 0.
ERC 0; DRC = 499 unrouted items only.

Generated with [Devin](https://devin.ai)

Co-Authored-By: Devin <158243242+devin-ai-integration[bot]@users.noreply.github.com>
Parts:
- added C85: 47u, Capacitor_SMD:C_0603_1608Metric, symbol vitalq:C
Connections:
- net GND: now also C85.2
- net VBAT: now also C85.1
