File: hardware/pcb/max86178.kicad_sch (KiCad schematic)
At the start: 24 parts, among them J10 Optical tail pads, J11 Sweat site, J12 FH12-14S, J13 MX ECG pads, J9 I2C tail pads, U22 MAX86178ENJ+

Commit message: Fit tier-1 DNP parts: U24 RTC, U25 mic, D26-D30 tail clamps
- U24 RV-3028-C7 + C77/R112/R115 support passives now fitted
- U25 IM69D130 PDM mic + C78 decoupling now fitted
- D26-D30 TPD1E10B06 tail ESD clamps now fitted
- remaining DNP are intentional options only: R61 cell-NTC,
  R104/R105 CP2102 USB strap, R107/R108 SPARE divider, J12, J13

check.sh PASS: ERC 0; gates 0; DRC = 499 unrouted items only.

Generated with [Devin](https://devin.ai)

Co-Authored-By: Devin <158243242+devin-ai-integration[bot]@users.noreply.github.com>
Parts:
- D26, D27, D28, D29, D30: now fitted
Other:
- note added: "J13 DNP pads: optional second ECG input pair. R118/R119 + D29/D30 fitted."
- note removed: "J13 DNP: optional second ECG input pair. R118/R119 + D29/D30 ladder footprints."
