File: hardware/pcb/mcu.kicad_sch (KiCad schematic)
At the start: 19 parts, among them J3 FSR pads, U1 ESP32-S3-MINI-1-N4R2, U18 W25Q512JVEIQ, U19 TCA6408ARSVR, U25 IM69D130

Commit message: Fit tier-1 DNP parts: U24 RTC, U25 mic, D26-D30 tail clamps
- U24 RV-3028-C7 + C77/R112/R115 support passives now fitted
- U25 IM69D130 PDM mic + C78 decoupling now fitted
- D26-D30 TPD1E10B06 tail ESD clamps now fitted
- remaining DNP are intentional options only: R61 cell-NTC,
  R104/R105 CP2102 USB strap, R107/R108 SPARE divider, J12, J13

check.sh PASS: ERC 0; gates 0; DRC = 499 unrouted items only.

Generated with [Devin](https://devin.ai)

Co-Authored-By: Devin <158243242+devin-ai-integration[bot]@users.noreply.github.com>
Parts:
- C78, U25: now fitted
Other:
- note added: "U25 IM69D130. PDM on IO40/IO41. 100 nF on VDD (datasheet)."
- note removed: "U25 IM69D130, DNP. PDM on IO40/IO41. 100 nF on VDD (datasheet)."
