File: hardware/pcb/vitalq_hw_v1_WIP.kicad_pcb (KiCad board)
At the start: 6 copper layers, 46 x 70 mm, 292 parts, among them J1 USB-C, J10 Optical tail pads, J11 Sweat site, J12 FH12-14S, J13 MX ECG pads, J2 LiPo pads, J3 FSR pads, J5 ECG pads, J6 EDA pads, J7 Chest bioZ, J8 TC2030, J9 I2C tail pads, Q1 CSD13380F3T, Q2 CSD13380F3T, Q3 BC847BS,115, Q4 CSD13380F3T, SW1 TS-1088, SW2 TS-1088, U1 ESP32-S3-MINI-1-N4R2, U10 AS7341-DLGM, U11 TMP117AIDRVR, U12 MLX90632SLD-DCB-100-SP, U13 BME280, U14 LSM6DSV80XTR, U15 TPS61240YFFR, U16 SFH 7072, U17 MAX17048G+T10, U18 W25Q512JVEIQ, U19 TCA6408ARSVR, U2 BQ25170DSGR, U20 TMP117AIDRVR, U21 USBLC6-2SC6, U22 MAX86178ENJ+, U23 SHT45-AD1B, U24 RV-3028-C7, U25 IM69D130, U3 TPS63802DLAR, U4 TPS7A2018PDBVR, U5 CP2102N-A02-GQFN28R, U6 AFE4900YZR, U7 AD5940BCBZ-RL7, U8 ADS1292RIRSMT, U9 PCA9306DCUR

Commit message: Route hw_v2 six-layer WIP: flood/BFS router, HV electrode corridor, liberate workers
Board grown to 46x70 with all 292 parts placed and placement gates clean.
~5,160 track segments + ~480 vias routed across F/B/In2/In3 (In1 held clear
by hv_inner creepage rule area; In4 is the power-plane pour layer).

New deterministic routing toolchain: obstacle index + 8-dir BFS flood with
via hops (route_all/route_flood), HV electrode emitters (emit_hv*, emit_one,
emit_drv), parallel worker sharding (worker_route + merge_workers), and a
surgical liberator (liberate.py) that censuses sealed-pad choke items,
performs bounded rip-up, and re-heals displaced nets. merge_delta replays
worker rip logs centrally.

State: vitalq_hw_v1_WIP.kicad_pcb is a reviewable WIP — ~35 nets verified
end-to-end; ~140 opens remain, concentrated on pads entombed by dense
copper inside/around the reserved electrode corridor (BFS saturates before
reaching them; even Freerouting's fanout stage plateaus on the same set).
NOT fabrication-ready: residual opens, DRC/ERC and zone-fill pass pending.

Generated with [Devin](https://devin.ai)

Co-Authored-By: Devin <158243242+devin-ai-integration[bot]@users.noreply.github.com>
Routing:
- net ECG1_PAD: track 3.97 -> 109.9 mm, vias 1 -> 3
- net SPI_SCK: track 9.06 -> 104.6 mm, vias 2 -> 9
- net ADS1292_DRDY: track 3.27 -> 92.5 mm, vias 1 -> 10
- net NIR730_GATE: track 2.75 -> 90.9 mm, vias 0 -> 6
- net EDA_SE_PAD: track 48.9 -> 135.6 mm, vias 2 -> 5
- net IR_K: track 2.87 -> 84.1 mm, vias 1 -> 6
- net IR_GATE: track 5.30 -> 75.3 mm, vias 1 -> 7
- net ECG2_PAD: track 21.9 -> 88.9 mm, vias 1 -> 3
- net I2C_SDA_1V8: track 13.5 -> 77.4 mm, vias 1 -> 4
- net EDA_DE_PAD: track 0.00 -> 63.6 mm, vias 1 -> 3
- net RLD_PAD: track 6.64 -> 67.6 mm, vias 0 -> 3
- net AFE_P_PAD: track 49.8 -> 99.1 mm, vias 1 -> 3
- net EDA_RE_PAD: track 43.9 -> 90.6 mm, vias 3 -> 4
- net RTC_INT: track 4.99 -> 45.7 mm, vias 0 -> 3
- net SWEAT_RE: track 113.2 -> 84.2 mm
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
Commit message: WIP sync: microvia escapes landing, ~101 nets closed this pass
Liberate now emits blind microvias (0.3mm/0.1mm drill) to free pocketed BGA
pads onto inner layers — the unlock for the entombed-pad class. converge.py
loops opens->liberate->verify autonomously.

Generated with [Devin](https://devin.ai)

Co-Authored-By: Devin <158243242+devin-ai-integration[bot]@users.noreply.github.com>
Routing:
- net TX4: track 22.2 -> 40.5 mm, vias 2 -> 3
- net +1V8: track 28.5 -> 46.2 mm
- net VBUS: track 53.9 -> 36.5 mm, vias 9 -> 10
- net SPI_SCK: track 104.6 -> 117.2 mm, vias 9 -> 10
- net ADS1292_PWDN: track 22.7 -> 11.2 mm, vias 3 -> 2
- net PD_K: track 79.9 -> 70.5 mm, vias 8 -> 6
- net AFE_N_AC: track 77.1 -> 67.9 mm
- net LED2_K: track 60.9 -> 53.1 mm, vias 4 -> 2
- net LED3_K: track 73.8 -> 66.3 mm, vias 5 -> 3
- net ECG_N: track 60.6 -> 53.2 mm
- net I2C_SDA: track 121.7 -> 115.2 mm
- net FN_SURGE: track 18.2 -> 11.8 mm, vias 4 -> 3
- net IR_GATE: track 75.3 -> 69.3 mm
- net +3V3_ANA: track 57.7 -> 51.8 mm, vias 8 -> 11
- net EXP_INT: track 28.7 -> 33.8 mm, vias 4 -> 5
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