File: hardware/pcb/vitalq_quilter_input.kicad_pcb (KiCad board)
At the start: 6 copper layers, 46 x 70 mm, 292 parts, among them J1 USB-C, J10 Optical tail pads, J11 Sweat site, J12 FH12-14S, J13 MX ECG pads, J2 LiPo pads, J3 FSR pads, J5 ECG pads, J6 EDA pads, J7 Chest bioZ, J8 TC2030, J9 I2C tail pads, Q1 CSD13380F3T, Q2 CSD13380F3T, Q3 BC847BS,115, Q4 CSD13380F3T, SW1 TS-1088, SW2 TS-1088, U1 ESP32-S3-MINI-1-N4R2, U10 AS7341-DLGM, U11 TMP117AIDRVR, U12 MLX90632SLD-DCB-100-SP, U13 BME280, U14 LSM6DSV80XTR, U15 TPS61240YFFR, U16 SFH 7072, U17 MAX17048G+T10, U18 W25Q512JVEIQ, U19 TCA6408ARSVR, U2 BQ25170DSGR, U20 TMP117AIDRVR, U21 USBLC6-2SC6, U22 MAX86178ENJ+, U23 SHT45-AD1B, U24 RV-3028-C7, U25 IM69D130, U3 TPS63802DLAR, U4 TPS7A2018PDBVR, U5 CP2102N-A02-GQFN28R, U6 AFE4900YZR, U7 AD5940BCBZ-RL7, U8 ADS1292RIRSMT, U9 PCA9306DCUR

Commit message: U22 MAX86178: real 49-ball WLP footprint + pin map from ADI/Ultra Librarian model; remap nets by function
Connections:
- U22 pad A1: PD_A -> unconnected-(U22-BIOZ_EL2A-PadA1)
- U22 pad A2: PD_K -> unconnected-(U22-BIOZ_EL3A-PadA2)
- U22 pad A3: LED1_K -> unconnected-(U22-BIOZ_EL1-PadA3)
- U22 pad A4: LED2_K -> unconnected-(U22-BIOZ_EL4-PadA4)
- U22 pad A5: LED3_K -> unconnected-(U22-CAL1-PadA5)
- U22 pad A6: MX_ECG_INP -> MX_ECG_INM
- U22 pad A7: MX_ECG_INM -> MX_ECG_INP
- U22 pad F1: +3V3_ANA -> unconnected-(U22-LED6_DRV-PadF1)
- U22 pad F2: +3V3 -> unconnected-(U22-LED4_DRV-PadF2)
- U22 pad F3: VBAT -> LED2_K
- U22 pad F4: MX_VREF -> MISO_MX
- U22 pad F5: GND -> unconnected-(U22-FCLK-PadF5)
- U22 pad F6: GND -> unconnected-(U22-VREF_ECG-PadF6)
- U22 pad F7: GND -> +3V3_ANA
- U22 pad G2: unconnected-(U22-RSV-PadG2) -> LED3_K
- U22 pad G3: MAX86178_INT -> LED1_K
- U22 pad G4: CS_MAX86178 -> MAX86178_INT
- U22 pad G5: MISO_MX -> unconnected-(U22-INT2-PadG5)
- U22 pad G6: SPI_MOSI -> unconnected-(U22-TRIG-PadG6)
- U22 pad G7: SPI_SCK -> +3V3
