File: hardware/pcb/vitalq_quilter_input.kicad_pcb (KiCad board)
At the start: 6 copper layers, 46 x 70 mm, 292 parts, among them J1 USB-C, J10 Optical tail pads, J11 Sweat site, J12 FH12-14S, J13 MX ECG pads, J2 LiPo pads, J3 FSR pads, J5 ECG pads, J6 EDA pads, J7 Chest bioZ, J8 TC2030, J9 I2C tail pads, Q1 CSD13380F3T, Q2 CSD13380F3T, Q3 BC847BS,115, Q4 CSD13380F3T, SW1 TS-1088, SW2 TS-1088, U1 ESP32-S3-MINI-1-N4R2, U10 AS7341-DLGM, U11 TMP117AIDRVR, U12 MLX90632SLD-DCB-100-SP, U13 BME280, U14 LSM6DSV80XTR, U15 TPS61240YFFR, U16 SFH 7072, U17 MAX17048G+T10, U18 W25Q512JVEIQ, U19 TCA6408ARSVR, U2 BQ25170DSGR, U20 TMP117AIDRVR, U21 USBLC6-2SC6, U22 MAX86178ENJ+, U23 SHT45-AD1B, U24 RV-3028-C7, U25 IM69D130, U3 TPS63802DLAR, U4 TPS7A2018PDBVR, U5 CP2102N-A02-GQFN28R, U6 AFE4900YZR, U7 AD5940BCBZ-RL7, U8 ADS1292RIRSMT, U9 PCA9306DCUR

Commit message: hw_v2.1: swap U22 MAX86178->MAX86141, add U26 level shifter + bypass caps
U22 is now MAX86141ENP+ (20-bump WLP, vitalq:MAX86141_WLP20): same
refdes, schematic/footprint UUIDs, and locked B.Cu position. SDO is
1.8 V, so new U26 SN74AXC2T245RSWR shifts it into MISO_MX with OE on
CS_MAX86178 (tri-state while deselected). C86-C91 added for U22/U26
rails. MAX86178 ECG/BioZ channels dropped; D29/D30/R118/R119 left in
place but now unused.

Netlist diff vs previous: only U22/U26/C86-C91 + new MX_SDO_1V8 net
changed, zero unexpected pin-to-net differences. Applied identically to
~/Downloads/VitalQ_Quilter_v5 (292->299 footprints, U22 20 pads,
schematic-parity DRC clean, ERC 0 errors) and mirrored into the flat
schematic + quilter input board here. Transform is scripted in
hardware/pcb/swap_max86141.py. Docs updated.

Generated with [Devin](https://devin.ai)

Co-Authored-By: Devin <158243242+devin-ai-integration[bot]@users.noreply.github.com>
Parts:
- added C86: 100n, Capacitor_SMD:C_0402_1005Metric, F.Cu at (65.0, 21.0)
- added C87: 10u, Capacitor_SMD:C_0402_1005Metric, F.Cu at (73.0, 21.0)
- added C88: 100n, Capacitor_SMD:C_0402_1005Metric, F.Cu at (81.0, 21.0)
- added C89: 10u, Capacitor_SMD:C_0603_1608Metric, B.Cu at (89.0, 21.0)
- added C90: 100n, Capacitor_SMD:C_0402_1005Metric, F.Cu at (97.0, 21.0)
- added C91: 100n, Capacitor_SMD:C_0402_1005Metric, F.Cu at (105.0, 21.0)
- added U26: SN74AXC2T245RSWR, Package_DFN_QFN:Texas_RSW0010A_UQFN-10_1.4x1.8mm_P0.4mm, F.Cu at (57.0, 21.0)
- U22: value MAX86178ENJ+ -> MAX86141ENP+; footprint vitalq:MAX86178_WLP49 -> vitalq:MAX86141_WLP20
Connections:
- U22 pad A1: unconnected-(U22-BIOZ_EL2A-PadA1) -> TX_5V
- U22 pad A2: unconnected-(U22-BIOZ_EL3A-PadA2) -> SPI_SCK
- U22 pad A3: unconnected-(U22-BIOZ_EL1-PadA3) -> MX_SDO_1V8
- U22 pad A4: unconnected-(U22-BIOZ_EL4-PadA4) -> SPI_MOSI
- U22 pad A5: unconnected-(U22-CAL1-PadA5) -> CS_MAX86178
- U22 pad B1: unconnected-(U22-BIOZ_EL2B-PadB1) -> LED3_K
- U22 pad B2: unconnected-(U22-BIOZ_EL3B-PadB2) -> MAX86178_INT
- U22 pad B5: unconnected-(U22-CAL2-PadB5) -> MX_VREF
- U22 pad C1: PD_K -> LED2_K
- U22 pad C2: unconnected-(U22-PD4_IN-PadC2) -> +1V8
- U22 pad C4: unconnected-(U22-DRVXR-PadC4) -> GND
- U22 pad C5: unconnected-(U22-DRVSJ-PadC5) -> PD_A
- U22 pad D1: unconnected-(U22-PD2_IN-PadD1) -> LED1_K
- U22 pad D2: unconnected-(U22-PD3_IN-PadD2) -> +1V8
- U22 pad D4: CS_MAX86178 -> unconnected-(U22-PD2_IN-PadD4)
- U22 pad D5: unconnected-(U22-DRVXC-PadD5) -> PD_K
