File: hardware/pcb/vitalq_quilter_input.kicad_pcb (KiCad board)
At the start: 6 copper layers, 46 x 70 mm, 299 parts, among them J1 USB-C, J10 Optical tail pads, J11 Sweat site, J12 FH12-14S, J13 MX ECG pads, J2 LiPo pads, J3 FSR pads, J5 ECG pads, J6 EDA pads, J7 Chest bioZ, J8 TC2030, J9 I2C tail pads, Q1 CSD13380F3T, Q2 CSD13380F3T, Q3 BC847BS,115, Q4 CSD13380F3T, SW1 TS-1088, SW2 TS-1088, U1 ESP32-S3-MINI-1-N4R2, U10 AS7341-DLGM, U11 TMP117AIDRVR, U12 MLX90632SLD-DCB-100-SP, U13 BME280, U14 LSM6DSV80XTR, U15 TPS61240YFFR, U16 SFH 7072, U17 MAX17048G+T10, U18 W25Q512JVEIQ, U19 TCA6408ARSVR, U2 BQ25170DSGR, U20 TMP117AIDRVR, U21 USBLC6-2SC6, U22 MAX86141ENP+, U23 SHT45-AD1B, U24 RV-3028-C7, U25 IM69D130, U26 SN74AXC2T245RSWR, U3 TPS63802DLAR, U4 TPS7A2018PDBVR, U5 CP2102N-A02-GQFN28R, U6 AFE4900YZR, U7 AD5940BCBZ-RL7, U8 ADS1292RIRSMT, U9 PCA9306DCUR

Commit message: pcb: enlarge outline 46x70 -> 50x75 for Quilter v7
Symmetric growth about board centre (23,27): x -2..48, y -10.5..64.5.
Skin-side sensor cluster + HV corridor + electrode pads shift +2.5mm Y
as one rigid group (same standoff from the +Y skin edge); tail pads
J9-J11 +2mm X and FFC J12 -2mm X to stay edge-flush; -Y end group
(J1 USB-C, U1 ESP32 + antenna keepout, J2) -2.5mm Y. H1/H2 returned
on-board at original corner insets and locked. Zones moved with their
groups; interior cutouts follow the cluster. Netlist diff vs v6: zero.
R122's 0.64mm edge overhang is pre-existing from v6, preserved.

Generated with [Devin](https://devin.ai)

Co-Authored-By: Devin <158243242+devin-ai-integration[bot]@users.noreply.github.com>
Parts:
- moved H2 180.8 mm to (-0.15, -7.18)
- moved H1 173.5 mm to (0.60, -2.19)
- moved J10 3.20 mm to (46.8, 45.9)
- moved J11 3.20 mm to (46.8, 57.5)
- moved J12 3.20 mm to (1.30, 52.5)
- moved J9 3.20 mm to (46.8, 17.5)
- moved D1 2.50 mm to (4.90, 22.5)
- moved D10 2.50 mm to (24.8, 57.5)
- moved D11 2.50 mm to (14.0, 48.8)
- moved D12 2.50 mm to (15.9, 50.8)
- moved D2 2.50 mm to (6.35, 22.5)
- moved D21 2.50 mm to (17.9, 22.5)
- moved D22 2.50 mm to (19.4, 22.5)
- moved D23 2.50 mm to (20.9, 22.7)
- moved D24 2.50 mm to (23.4, 22.9)
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Other:
- board size 46 x 70 mm -> 50 x 75 mm
