File: hardware/pcb/vitalq_flat.kicad_sch (KiCad schematic)
At the start: 292 parts, among them J1 USB-C, J10 Optical tail pads, J11 Sweat site, J12 FH12-14S, J13 MX ECG pads, J2 LiPo pads, J3 FSR pads, J5 ECG pads, J6 EDA pads, J7 Chest bioZ, J8 TC2030, J9 I2C tail pads, Q1 CSD13380F3T, Q2 CSD13380F3T, Q3 BC847BS,115, Q4 CSD13380F3T, SW1 TS-1088, SW2 TS-1088, U1 ESP32-S3-MINI-1-N4R2, U10 AS7341-DLGM, U11 TMP117AIDRVR, U12 MLX90632SLD-DCB-100-SP, U13 BME280, U14 LSM6DSV80XTR, U15 TPS61240YFFR, U16 SFH 7072, U17 MAX17048G+T10, U18 W25Q512JVEIQ, U19 TCA6408ARSVR, U2 BQ25170DSGR, U20 TMP117AIDRVR, U21 USBLC6-2SC6, U22 MAX86178ENJ+, U23 SHT45-AD1B, U24 RV-3028-C7, U25 IM69D130, U3 TPS63802DLAR, U4 TPS7A2018PDBVR, U5 CP2102N-A02-GQFN28R, U6 AFE4900YZR, U7 AD5940BCBZ-RL7, U8 ADS1292RIRSMT, U9 PCA9306DCUR

Commit message: hw_v2.1: swap U22 MAX86178->MAX86141, add U26 level shifter + bypass caps
U22 is now MAX86141ENP+ (20-bump WLP, vitalq:MAX86141_WLP20): same
refdes, schematic/footprint UUIDs, and locked B.Cu position. SDO is
1.8 V, so new U26 SN74AXC2T245RSWR shifts it into MISO_MX with OE on
CS_MAX86178 (tri-state while deselected). C86-C91 added for U22/U26
rails. MAX86178 ECG/BioZ channels dropped; D29/D30/R118/R119 left in
place but now unused.

Netlist diff vs previous: only U22/U26/C86-C91 + new MX_SDO_1V8 net
changed, zero unexpected pin-to-net differences. Applied identically to
~/Downloads/VitalQ_Quilter_v5 (292->299 footprints, U22 20 pads,
schematic-parity DRC clean, ERC 0 errors) and mirrored into the flat
schematic + quilter input board here. Transform is scripted in
hardware/pcb/swap_max86141.py. Docs updated.

Generated with [Devin](https://devin.ai)

Co-Authored-By: Devin <158243242+devin-ai-integration[bot]@users.noreply.github.com>
Parts:
- added C86, C88, C90, C91: 100n, Capacitor_SMD:C_0402_1005Metric, symbol vitalq:C
- added C87: 10u, Capacitor_SMD:C_0402_1005Metric, symbol vitalq:C
- added C89: 10u, Capacitor_SMD:C_0603_1608Metric, symbol vitalq:C
- added U26: SN74AXC2T245RSWR, Package_DFN_QFN:Texas_RSW0010A_UQFN-10_1.4x1.8mm_P0.4mm, symbol vitalq:SN74AXC2T245
- U22: value MAX86178ENJ+ -> MAX86141ENP+; footprint vitalq:MAX86178_WLP49 -> vitalq:MAX86141_WLP20; symbol vitalq:MAX86178 -> vitalq:MAX86141; LCSC (none) -> C5328762
Connections:
- net +1V8: now also U22.C2 (VDD_DIG), U22.D2 (VDD_ANA), C86.1, C87.1, C88.1, C90.1, U26.10 (DIR1), U26.7 (VCCA)
- net +3V3: now also C91.1, U26.6 (VCCB); no longer U22.G7 (IOVDD)
- net +3V3_ANA: no longer U22.F7 (LDO_IN)
- net CS_MAX86178: now also U22.A5 (CSB), U26.2 (OE); no longer U22.D4 (CSB/I2C_SEL)
- net GND: now also U22.C4 (GND_ANA), C86.2, C87.2, C88.2, C89.2, C90.2, C91.2, U26.1 (DIR2), U26.3 (GND), U26.4 (B2); no longer U22.E1 (PGND)
- net LED1_K: now also U22.D1 (LED1_DRV); no longer U22.G3 (LED1_DRV)
- net LED2_K: now also U22.C1 (LED2_DRV); no longer U22.F3 (LED2_DRV)
- net LED3_K: now also U22.B1 (LED3_DRV); no longer U22.G2 (LED3_DRV)
- net MAX86178_INT: now also U22.B2 (INT); no longer U22.G4 (INT1)
- net MISO_MX: now also U26.5 (B1); no longer U22.F4 (SDO/ADDR)
- net MX_ECG_INM: no longer U22.A6 (ECG_EL2)
- net MX_ECG_INP: no longer U22.A7 (ECG_EL1)
- net MX_VREF: now also U22.B5 (VREF); no longer U22.E2 (VREF_PPG)
- net PD_A: now also U22.C5 (PD_GND)
- net PD_K: now also U22.D5 (PD1_IN); no longer U22.C1 (PD1_IN)
- net SPI_MOSI: now also U22.A4 (SDI); no longer U22.E5 (SDI/SDA)
- net SPI_SCK: now also U22.A2 (SCLK); no longer U22.E4 (SCLK/SCL)
- net TX_5V: now also U22.A1 (VLED), C89.1
- net VBAT: no longer U22.E3 (VLED)
- net MX_SDO_1V8: now reaches U22.A3 (SDO)
- net MX_SDO_1V8: now also U26.8 (A1)
- removed net AVDD: U22.D6 (AVDD)
- removed net DVDD: U22.D7 (DVDD)
- removed net LDO_OUT: U22.E7 (LDO_OUT)
- no-connect marks 52 -> 56
