File: hardware/pcb/vitalq_v2.kicad_pcb (KiCad board)
At the start: 8 copper layers, 55.6 x 75 mm, 302 parts, among them J1 USB-C, J10 Optical tail pads, J11 Sweat site, J12 FH12-14S, J13 MX ECG pads, J2 LiPo pads, J3 FSR pads, J5 ECG pads, J6 EDA pads, J7 Chest bioZ, J8 TC2030, J9 I2C tail pads, Q1 CSD13380F3T, Q2 CSD13380F3T, Q3 BC847BS,115, Q4 CSD13380F3T, Q6 AO3401A, SW1 TS-1088, SW2 TS-1088, U1 ESP32-S3-MINI-1-N4R2, U10 AS7341-DLGM, U11 TMP117AIDRVR, U12 MLX90632SLD-DCB-100-SP, U13 BME280, U14 LSM6DSV80XTR, U15 TPS61240YFFR, U16 SFH 7072, U17 MAX17048G+T10, U18 W25Q512JVEIQ, U19 TCA6408ARSVR, U2 BQ25170DSGR, U20 TMP117AIDRVR, U21 USBLC6-2SC6, U22 MAX86141ENP+, U23 SHT45-AD1B, U24 RV-3028-C7, U25 IM69D130, U26 SN74AXC2T245RSWR, U3 TPS63802DLAR, U4 TPS7A2018PDBVR, U5 CP2102N-A02-GQFN28R, U6 AFE4900YZR, U7 AD5940BCBZ-RL7, U8 ADS1292RIRSMT, U9 PCA9306DCUR

Commit message: pcb fix_v19a: U15 paste, U14 transpose, R61 DNP, TPS61241, fp fixes, mic R-slot
Board+lib: U14/U8/U19/U26/U9/U11/U4 pad corrections (pos gaps verified).
Gerber: F_Paste +6 flashes @U15 (54%->84% coverage). BOM/CPL: R61 DNP,
U15->TPS61241YFFR C544431. Docs: POFV-48 list, provenance. FW: IM69D130
decodes RIGHT slot (SELECT=GND, DSR_16S inversion) — sim mic_pdm PASS.

Generated with [Devin](https://devin.ai)
Parts:
- D10: value JB3030UWT-B-H50EA0000-1Z000001 -> NF2W757G-F1
