File: hardware/pcb/vitalquant_v2.kicad_pcb (KiCad board)
At the start: 8 copper layers, 55.6 x 81 mm, 302 parts, among them J1 USB-C, J10 Optical tail pads, J11 Sweat site, J12 FH12-14S, J13 MX ECG pads, J2 LiPo pads, J3 FSR pads, J5 ECG pads, J6 EDA pads, J7 Chest bioZ, J8 TC2030, J9 I2C tail pads, Q1 CSD13380F3T, Q2 CSD13380F3T, Q3 BC847BS,115, Q4 CSD13380F3T, Q6 AO3401A, SW1 TS-1088, SW2 TS-1088, U1 ESP32-S3-WROOM-1-N16R8, U10 AS7341-DLGM, U11 TMP117AIDRVR, U12 MLX90632SLD-DCB-100-RE, U13 BME280, U14 LSM6DSV320XTR, U15 TPS61240YFFR, U16 SFH 7072, U17 MAX17048G+T10, U18 W25Q512JVEIQ, U19 TCA6408ARSVR, U2 BQ25170DSGR, U20 TMP117AIDRVR, U21 USBLC6-2SC6, U22 MAX86141ENP+, U23 SHT45-AD1B, U24 RV-3028-C7, U25 IM69D130, U26 SN74AXC2T245RSWR, U3 TPS63802DLAR, U4 TPS7A2018PDBVR, U5 CP2102N-A02-GQFN28R, U6 AFE4900YZR, U7 AD5940BCBZ-RL7, U8 ADS1292RIRSMR, U9 PCA9306DCUR

Commit message: hw(pcb): fix_v25 - 12 test points + bring-up plan, no existing copper moved
Test-point revision on the fix_v24 design (KiCad 10.0.4):
- TP29-TP40, all on F.Cu (top/lid side), TestPoint_Pad_D1.0mm, each with
  a short 0.15 mm stub to existing same-net copper; no vias needed
- Nets: RLDREF, RLDOUT, VBAT_SYS, +3V3_ANA, TX_5V_RAW, RTC_VBK,
  +3V3_ESP, IOVDD, CHG_ISET, CHG_VSET, VBUS_DET, TS - covering the
  AFE/ADC reference and power-path nodes the spec asked for on top of
  TP1-TP28 (which already cover rails, GND, UART, boot straps, I2C, SPI)
- Skipped and logged: AFE_BG/AVDD_REG/DVDD_REG/VREF2/CHG_PG (no DRC-safe
  free copper), USB_DP/USB_DM (UART TPs exist; pad capacitance on a
  480 Mb/s pair; R104/R105 DNP anyway)
- Schematic parity: matching vitalquant:TestPoint symbols + labels added
- All new TPs: DNP, in_bom=no, exclude_from_bom + exclude_from_pos_files;
  grep-verified absent from BOM.csv/BOM_JLC/CPL/CPL_JLC/positions
- UUID-keyed diff vs fix_v24: 0 pre-existing items changed
  (reports/COPPER_DIFF_V25.txt); drill holes identical (917 PTH + 8 NPTH)
- DRC --severity-error --schematic-parity: 0 violations / 0 unconnected /
  0 shorts / 0 parity issues; ERC --severity-error: 0 violations
- reports/: BRINGUP.md (first-power-on plan), REPORT_V25.md,
  COPPER_DIFF_V25.txt; fab/ regenerated (gerbers, jlc, drill, assembly,
  zips, notes, verification, checksums); ci.yml zip name -> fixv25

Based on branch fix/bom-v24 (PR #19 head, commit 842de500).

Generated with [Devin](https://devin.ai)

Co-Authored-By: Devin <158243242+devin-ai-integration[bot]@users.noreply.github.com>
Parts:
- added TP29: RLDREF, TestPoint:TestPoint_Pad_D1.0mm, F.Cu at (46.9, 7.60)
- added TP30: RLDOUT, TestPoint:TestPoint_Pad_D1.0mm, F.Cu at (48.2, 28.6)
- added TP31: VBAT_SYS, TestPoint:TestPoint_Pad_D1.0mm, F.Cu at (46.6, 26.3)
- added TP32: +3V3_ANA, TestPoint:TestPoint_Pad_D1.0mm, F.Cu at (42.6, 7.12)
- added TP33: TX_5V_RAW, TestPoint:TestPoint_Pad_D1.0mm, F.Cu at (40.2, 41.4)
- added TP34: RTC_VBK, TestPoint:TestPoint_Pad_D1.0mm, F.Cu at (29.7, 22.3)
- added TP35: +3V3_ESP, TestPoint:TestPoint_Pad_D1.0mm, F.Cu at (1.52, 10.8)
- added TP36: IOVDD, TestPoint:TestPoint_Pad_D1.0mm, F.Cu at (45.0, -9.44)
- added TP37: CHG_ISET, TestPoint:TestPoint_Pad_D1.0mm, F.Cu at (26.8, 10.8)
- added TP38: CHG_VSET, TestPoint:TestPoint_Pad_D1.0mm, F.Cu at (29.9, 10.6)
- added TP39: VBUS_DET, TestPoint:TestPoint_Pad_D1.0mm, F.Cu at (4.80, 57.0)
- added TP40: TS, TestPoint:TestPoint_Pad_D1.0mm, F.Cu at (28.9, 8.00)
Routing:
- net +3V3_ANA: track 146.3 -> 148.5 mm
- net VBUS_DET: track 62.0 -> 64.0 mm
- net TX_5V_RAW: track 26.4 -> 28.4 mm
- net RLDREF: track 17.6 -> 19.4 mm
- net CHG_VSET: track 33.0 -> 34.5 mm
- net +3V3_ESP: track 88.0 -> 89.3 mm
- net TS: track 29.7 -> 30.9 mm
- net RLDOUT: track 110.8 -> 112.1 mm
- net IOVDD: track 47.5 -> 48.1 mm
- net VBAT_SYS: track 15.3 -> 15.9 mm
- net CHG_ISET: track 18.2 -> 18.8 mm
