File: hardware/pcb/kicad/vitalq_v2.kicad_sch (KiCad schematic)
At the start: 302 parts, among them J1 USB-C, J10 Optical tail pads, J11 Sweat site, J12 FH12-14S, J13 MX ECG pads, J2 LiPo pads, J3 FSR pads, J5 ECG pads, J6 EDA pads, J7 Chest bioZ, J8 TC2030, J9 I2C tail pads, Q1 CSD13380F3T, Q2 CSD13380F3T, Q3 BC847BS,115, Q4 CSD13380F3T, Q6 AO3401A, SW1 TS-1088, SW2 TS-1088, U1 ESP32-S3-WROOM-1-N16R8, U10 AS7341-DLGM, U11 TMP117AIDRVR, U12 MLX90632SLD-DCB-100-SP, U13 BME280, U14 LSM6DSV80XTR, U15 TPS61240YFFR, U16 SFH 7072, U17 MAX17048G+T10, U18 W25Q512JVEIQ, U19 TCA6408ARSVR, U2 BQ25170DSGR, U20 TMP117AIDRVR, U21 USBLC6-2SC6, U22 MAX86141ENP+, U23 SHT45-AD1B, U24 RV-3028-C7, U25 IM69D130, U26 SN74AXC2T245RSWR, U3 TPS63802DLAR, U4 TPS7A2018PDBVR, U5 CP2102N-A02-GQFN28R, U6 AFE4900YZR, U7 AD5940BCBZ-RL7, U8 ADS1292RIRSMT, U9 PCA9306DCUR

Commit message: hw(pcb): fix_v23 board + corrected fab package
- Resolve the 10 KiCad 10.0.4 DRC errors measured on the reviewer run:
  9x Q1/Q2/Q4 intra-footprint pad clearances (0.100 mm TI PicoStar land
  pattern, scoped 0.09 mm rule in vitalq_v2.kicad_dru — matches JLCPCB
  multilayer minimum) and 1x J8 NPTH vs U6 courtyard (courtyard edge
  narrowed 1.30 -> 1.15 mm; hole stays 0.265 mm off the package body).
- Update schematic LCSC fields to the corrected 22 Oct BOM
  (U1 = ESP32-S3-WROOM-1-N16R8 C2913202, 37 refs + D10 C17610390);
  J12/U24/U25 excluded from JLC assembly files as DNP per main.
- Regenerate gerbers, drills, BOM/CPL, checksums and the fixv23
  fabrication zip; add reports/ VERIFY/DRC_STATEMENT/BOM_CROSSCHECK.
- DRC --severity-error --schematic-parity: 0/0/0; ERC: 0.

Co-Authored-By: Devin <158243242+devin-ai-integration[bot]@users.noreply.github.com>
Parts:
- C1, C47: LCSC C23124 -> C1705
- C21, C22, C23, C55, C68, C69, C70: LCSC C15115 -> C188347
- C34: LCSC C23692 -> C6261448
- C45, C7: LCSC C23677 -> C86295
- C46: LCSC C49240 -> C444845
- C63, C79: LCSC C14445 -> C52923
- C85: LCSC C23230 -> C730416
- C9: LCSC C307415 -> C15525
- D10: LCSC (none) -> C17610390
- R30, R31: LCSC C17275 -> C25893
- R32, R33, R34, R35, R36, R76, R77, R78, R79, R80, R81, R82, R83: LCSC C146900 -> C18009
- R43, R45: LCSC C283954 -> C3017614
- U1: LCSC C3013941 -> C2913202
- U18: LCSC C2986165 -> C7389628
- U23: LCSC C6705435 -> C5221601
Changed lines of the file:
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@@
 			)
 		)
-		(property "LCSC" "C23230"
+		(property "LCSC" "C730416"
 			(at 261.62 154.94 0)
 			(hide yes)
@@
 			)
 		)
-		(property "LCSC" "C146900"
+		(property "LCSC" "C18009"
 			(at 1270 674.37 0)
 			(hide yes)
@@
 			)
 		)
-		(property "LCSC" "C283954"
+		(property "LCSC" "C3017614"
 			(at 1884.68 233.68 0)
 			(hide yes)
@@
 			)
 		)
-		(property "LCSC" "C23124"
+		(property "LCSC" "C1705"
 			(at 1664.97 233.68 0)
 			(hide yes)
@@
 			)
 		)
-		(property "LCSC" "C146900"
+		(property "LCSC" "C18009"
 			(at 674.37 648.97 0)
 			(hide yes)
@@
 			)
 		)
-		(property "LCSC" "C146900"
+		(property "LCSC" "C18009"
 			(at 674.37 626.11 0)
 			(hide yes)
@@
 			)
 		)
-		(property "LCSC" "C146900"
+		(property "LCSC" "C18009"
 			(at 704.85 552.45 0)
 			(hide yes)
@@
 			)
 		)
-		(property "LCSC" "C23692"
+		(property "LCSC" "C6261448"
 			(at 1104.9 626.11 0)
 			(hide yes)
@@
 			)
 		)
-		(property "LCSC" "C3013941"
+		(property "LCSC" "C2913202"
 			(at 1184.91 123.19 0)
 			(hide yes)
@@
 			)
 		)
-		(property "LCSC" "C23677"
+		(property "LCSC" "C86295"
 			(at 1089.66 41.91 0)
 			(hide yes)
@@
 			)
 		)
-		(property "LCSC" "C23124"
+		(property "LCSC" "C1705"
 			(at 229.87 154.94 0)
 			(hide yes)
@@
 			)
 		)
-		(property "LCSC" "C14445"
+		(property "LCSC" "C52923"
 			(at 1285.24 919.48 0)
 			(hide yes)
@@
 			)
 		)
-		(property "LCSC" "C15115"
+		(property "LCSC" "C188347"
 			(at 815.34 574.04 0)
 			(hide yes)
@@
 			)
 		)
-		(property "LCSC" "C6705435"
+		(property "LCSC" "C5221601"
 			(at 1959.61 591.82 0)
 			(hide yes)
@@
 			)
 		)
-		(property "LCSC" "C17275"
+		(property "LCSC" "C25893"
 			(at 1365.25 661.67 0)
 			(hide yes)
@@
 			)
 		)
-		(property "LCSC" "C15115"
+		(property "LCSC" "C188347"
 			(at 815.34 552.45 0)
 			(hide yes)
@@
 			)
 		)
-		(property "LCSC" "C14445"
+		(property "LCSC" "C52923"
 			(at 596.9 53.34 0)
 			(hide yes)
@@
 			)
 		)
-		(property "LCSC" "C146900"
+		(property "LCSC" "C18009"
 			(at 1210.31 694.69 0)
 			(hide yes)
@@
 			)
 		)
-		(property "LCSC" "C146900"
+		(property "LCSC" "C18009"
 			(at 704.85 530.86 0)
 			(hide yes)
@@
 			)
 		)
-		(property "LCSC" "C15115"
+		(property "LCSC" "C188347"
 			(at 779.78 648.97 0)
 			(hide yes)
@@
 			)
 		)
-		(property "LCSC" "C23677"
+		(property "LCSC" "C86295"
 			(at 364.49 154.94 0)
 			(hide yes)
@@
 			)
 		)
-		(property "LCSC" "C15115"
+		(property "LCSC" "C188347"
 			(at 514.35 579.12 0)
 			(hide yes)
@@
 			)
 		)
-		(property "LCSC" "C15115"
+		(property "LCSC" "C188347"
 			(at 537.21 579.12 0)
 			(hide yes)
@@
 			)
 		)
-		(property "LCSC" "C17275"
+		(property "LCSC" "C25893"
 			(at 1295.4 661.67 0)
 			(hide yes)
@@
 			)
 		)
-		(property "LCSC" "C15115"
+		(property "LCSC" "C188347"
 			(at 815.34 596.9 0)
 			(hide yes)
@@
 			)
 		)
-		(property "LCSC" "C146900"
+		(property "LCSC" "C18009"
 			(at 1150.62 674.37 0)
 			(hide yes)
@@
 			)
 		)
-		(property "LCSC" "C146900"
+		(property "LCSC" "C18009"
 			(at 704.85 574.04 0)
 			(hide yes)
@@
 			)
 		)
-		(property "LCSC" "C146900"
+		(property "LCSC" "C18009"
 			(at 784.86 670.56 0)
 			(hide yes)
@@
 			)
 		)
-		(property "LCSC" "C146900"
+		(property "LCSC" "C18009"
 			(at 1089.66 674.37 0)
 			(hide yes)
@@
 			)
 		)
-		(property "LCSC" "C49240"
+		(property "LCSC" "C444845"
 			(at 1634.49 233.68 0)
 			(hide yes)
@@
 			)
 		)
-		(property "LCSC" "C307415"
+		(property "LCSC" "C15525"
 			(at 529.59 53.34 0)
 			(hide yes)
@@
 			)
 		)
-		(property "LCSC" "C283954"
+		(property "LCSC" "C3017614"
 			(at 1845.31 233.68 0)
 			(hide yes)
@@
 			)
 		)
-		(property "LCSC" "C2986165"
+		(property "LCSC" "C7389628"
 			(at 1104.9 233.68 0)
 			(hide yes)
@@
 			)
 		)
-		(property "LCSC" "C15115"
+		(property "LCSC" "C188347"
 			(at 624.84 541.02 0)
 			(hide yes)
@@
 			)
 		)
-		(property "LCSC" ""
+		(property "LCSC" "C17610390"
 			(at 1649.73 681.99 0)
 			(hide yes)
@@
 			)
 		)
-		(property "LCSC" "C146900"
+		(property "LCSC" "C18009"
 			(at 704.85 596.9 0)
 			(hide yes)
@@
 			)
 		)
-		(property "LCSC" "C146900"
+		(property "LCSC" "C18009"
 			(at 1329.69 674.37 0)
 			(hide yes)
@@
 			)
 		)
-		(property "LCSC" "C146900"
+		(property "LCSC" "C18009"
 			(at 674.37 670.56 0)
 			(hide yes)
